File: schematic/pi-pico-vga.kicad_sch (KiCad schematic)
At the start: 21 parts, among them J1 VGA, J2 PS/2, J3 Micro_SD_Card, Q1 2N7000, Q2 2N7000, SW1 RESET

Commit message: .
Parts:
- removed J2: PS/2, symbol Connector_Generic:Conn_01x06
- removed Q1, Q2: 2N7000, Package_TO_SOT_THT:TO-92_Inline, symbol Transistor_FET:2N7000
- removed R10, R11, R8, R9: 10K, symbol Device:R
- removed SW1: RESET, symbol Switch:SW_Push
Connections:
- net GPIO08: no longer names the net of A1.11 (GPIO8)
- net GPIO09: no longer names the net of A1.12 (GPIO9)
- no-connect marks 9 -> 7

Commit message: .
Parts:
- added BT1: Battery_Cell, symbol Device:Battery_Cell
- added C1: 0.1uF, symbol Device:C
- added C2: 10uF, symbol Device:C_Polarized
- added D3: LED, symbol Device:LED
- added J2: USB Keyboard, symbol Connector:USB_A
- added J4: Power, symbol Connector:USB_C_Receptacle_PowerOnly_6P
- added J5: UART, symbol Connector_Generic:Conn_01x06
- added J6: External, symbol Connector_Generic:Conn_02x05_Counter_Clockwise
- added J7: Jack-DC, symbol Connector:Jack-DC
- added R8: R, symbol Device:R
- added R9: 1k, symbol Device:R
- added RV2: 10k, symbol Device:R_Potentiometer
- added SW1: Power switch, symbol Switch:SW_SPST
- added SW2: User, symbol Switch:SW_Push
- added U1: DS1307+, Package_DIP:DIP-8_W7.62mm, symbol Timer_RTC:DS1307+
- added Y1: 32.768 Hz, symbol Device:Crystal
Connections:
- net +3.3V: now also J6.9 (Pin_9)
- net +5V: now also D3.2 (A), J2.1 (VBUS), J4.A9 (VBUS), J4.B9 (VBUS), J5.4 (Pin_4), J6.10 (Pin_10), U1.8 (VCC)
- net GND: now also C1.2, J2.4 (GND), J2.5 (Shield), J5.6 (Pin_6), J6.6 (Pin_6), J7.2, R8.1, RV2.3, SW1.2 (B), SW2.1
- net MISO: now also A1.6 (GPIO4), J6.2 (Pin_2); no longer A1.16 (GPIO12), J3.7 (DAT0)
- net MOSI: now also A1.5 (GPIO3), J6.1 (Pin_1); no longer A1.15 (GPIO11), J3.2 (DAT3/CD)
- net TX_PICO: now reaches A1.1 (GPIO0)
- net TX_PICO: now also J5.2 (Pin_2), J6.8 (Pin_8)
- net AUDIO: now reaches A1.10 (GPIO7)
- net AUDIO: now also R9.1
- net at A1.11 (GPIO8): now also U1.5 (SDA)
- net at A1.12 (GPIO9): now also U1.6 (SCL)
- net RX_PICO: now reaches A1.2 (GPIO1)
- net RX_PICO: now also J5.3 (Pin_3), J6.7 (Pin_7)
- net at A1.20 (GPIO15): now also SW2.2
- net SCK: now reaches A1.4 (GPIO2)
- net SCK: now also J6.3 (Pin_3)
- net CS0: now reaches A1.7 (GPIO5)
- net CS0: now also J6.4 (Pin_4)
- net USR0: now reaches A1.9 (GPIO6)
- net USR0: now also J6.5 (Pin_5)
- net CLK renamed SD_CLK
- net CS renamed SD_CS
- new net: D3.1 (K), R8.2
- new net: J4.A12 (GND), J4.B12 (GND), J4.S1 (SHIELD), SW1.1 (A)
- new net: C1.1, R9.2, RV2.1
- new net: C2.1, RV2.2
- new net: U1.1 (X1), Y1.1
- new net: U1.2 (X2), Y1.2
- new net: BT1.1 (+), U1.3 (VBAT)
- new net: BT1.2 (-), U1.4 (GND)
- new net: C2.2, J7.1
- new net PICO USB: J2.2 (D-), J2.3 (D+)
- new net SD_MISO: A1.16 (GPIO12), J3.7 (DAT0)
- new net SD_MOSI: A1.15 (GPIO11), J3.2 (DAT3/CD)
- no-connect marks 7 -> 14

Commit message: .
Connections:
- net +5V: now also A1.40 (VBUS); no longer A1.39 (VSYS)
- no-connect marks 14 -> 15
Changed lines of the file:
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@@
 	)
 	(no_connect
+		(at 120.65 60.96)
+	)
+	(no_connect
 		(at 222.25 134.62)
 	)
@@
 	(wire
 		(pts
+			(xy 125.73 59.69) (xy 125.73 60.96)
+		)
+		(stroke
+			(width 0)
+			(type default)
+		)
+	)
+	(wire
+		(pts
 			(xy 218.44 111.76) (xy 222.25 111.76)
 		)
@@
 	(wire
 		(pts
-			(xy 120.65 59.69) (xy 120.65 60.96)
-		)
-		(stroke
-			(width 0)
-			(type default)
-		)
-	)
-	(wire
-		(pts
 			(xy 176.53 105.41) (xy 182.88 105.41)
 		)
@@
 	(symbol
 		(lib_id "power:+5V")
-		(at 120.65 59.69 0)
+		(at 125.73 59.69 0)
 		(unit 1)
 		(exclude_from_sim no)
@@
 		(dnp no)
 		(property "Reference" "#PWR019"
-			(at 120.65 63.5 0)
+			(at 125.73 63.5 0)
 			(effects
 				(font
@@
 		)
 		(property "Value" "+5V"
-			(at 116.84 58.928 0)
+			(at 121.92 58.928 0)
 			(effects
 				(font
@@
 		)
 		(property "Footprint" ""
-			(at 120.65 59.69 0)
+			(at 125.73 59.69 0)
 			(effects
 				(font
@@
 		)
 		(property "Datasheet" ""
-			(at 120.65 59.69 0)
+			(at 125.73 59.69 0)
 			(effects
 				(font
@@
 		)
 		(property "Description" "Power symbol creates a global label with name \"+5V\""
-			(at 120.65 59.69 0)
+			(at 125.73 59.69 0)
 			(effects
 				(font

Commit message: .
Parts:
- added D4: LED, symbol Device:LED
- added R10: 220, symbol Device:R
- added SW3: SW_DIP_x02, symbol Switch:SW_DIP_x02
Connections:
- net GND: now also R10.2, SW3.3, SW3.4
- net at A1.19 (GPIO14): now also D4.2 (A)
- net at A1.32 (GPIO27_ADC1): now also SW3.1
- net at A1.34 (GPIO28_ADC2): now also SW3.2
- new net: D4.1 (K), R10.1
- no-connect marks 15 -> 18
Other:
- moved on the sheet: SW2

Commit message: .
Parts:
- added U2: Level Shift, Package_SO:SOIC-14_3.9x8.7mm_P1.27mm, symbol Logic_LevelTranslator:TXS0104ED
- SW3: value SW_DIP_x02 -> Microdip
Connections:
- net +3.3V: now also U2.9 (L_{VCC})
- net +5V: now also U2.3 (H_{VCC})
- net GND: now also SW2.2, U2.10 (GND), U2.4 (GND); no longer SW2.1
- net at A1.20 (GPIO15): now also SW2.1; no longer SW2.2
- net at U1.5 (SDA): now also U2.2 (H2); no longer A1.11 (GPIO8)
- net at U1.6 (SCL): now also U2.1 (H1); no longer A1.12 (GPIO9)
- new net SCL: A1.12 (GPIO9), U2.12 (L1)
- new net SDA: A1.11 (GPIO8), U2.11 (L2)
- no-connect marks 18 -> 23
Other:
- note added: "<- Notch"
- note added: "AUDIO"
- note added: "EXTERNAL INTERFACE"
- note added: "POWER"
- note added: "RTC"
- note added: "STORAGE"
- note added: "UART"
- note added: "USB INTERFACE"
- note added: "USER PANEL"
- note added: "VGA"
- moved on the sheet: BT1, C1, C2, D1, D2, D4, J1, J2, J3, J5, J6, J7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

Commit message: .
Parts:
- SW3: value Microdip -> Microswitch
Changed lines of the file:
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@@
 			)
 		)
-		(property "Value" "Microdip"
+		(property "Value" "Microswitch"
 			(at 132.08 146.05 0)
 			(effects

Commit message: .
Other:
- note added: "Notch ->"
- note removed: "<- Notch"
- moved on the sheet: J6
Changed lines of the file:
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@@
 	(text "EXTERNAL\nINTERFACE"
 		(exclude_from_sim no)
-		(at 115.57 191.008 0)
+		(at 133.35 189.738 0)
 		(effects
 			(font
@@
 		)
 	)
-	(text "<- Notch"
+	(text "USER\nPANEL"
 		(exclude_from_sim no)
-		(at 108.458 182.88 0)
+		(at 110.236 159.512 0)
 		(effects
 			(font
-				(size 1.27 1.27)
-				(thickness 0.254)
+				(size 2.54 2.54)
+				(thickness 0.508)
 				(bold yes)
 			)
 		)
 	)
-	(text "USER\nPANEL"
+	(text "Notch ->"
 		(exclude_from_sim no)
-		(at 110.236 159.512 0)
+		(at 83.058 181.864 0)
 		(effects
 			(font
-				(size 2.54 2.54)
-				(thickness 0.508)
+				(size 1.27 1.27)
+				(thickness 0.254)
 				(bold yes)
 			)
@@
 	(wire
 		(pts
-			(xy 102.87 175.26) (xy 102.87 180.34)
+			(xy 120.65 173.99) (xy 120.65 179.07)
 		)
 		(stroke
@@
 	(wire
 		(pts
-			(xy 102.87 180.34) (xy 92.71 180.34)
+			(xy 120.65 179.07) (xy 110.49 179.07)
 		)
 		(stroke
@@
 	(wire
 		(pts
-			(xy 95.25 177.8) (xy 92.71 177.8)
+			(xy 113.03 176.53) (xy 110.49 176.53)
 		)
 		(stroke
@@
 	(wire
 		(pts
-			(xy 71.12 180.34) (xy 80.01 180.34)
+			(xy 88.9 179.07) (xy 97.79 179.07)
 		)
 		(stroke
@@
 	(wire
 		(pts
-			(xy 71.12 177.8) (xy 80.01 177.8)
+			(xy 88.9 176.53) (xy 97.79 176.53)
 		)
 		(stroke
@@
 	(wire
 		(pts
-			(xy 95.25 190.5) (xy 95.25 187.96)
+			(xy 113.03 189.23) (xy 113.03 186.69)
 		)
 		(stroke
@@
 	(wire
 		(pts
-			(xy 71.12 182.88) (xy 80.01 182.88)
+			(xy 88.9 181.61) (xy 97.79 181.61)
 		)
 		(stroke
@@
 	(wire
 		(pts
-			(xy 95.25 175.26) (xy 95.25 177.8)
+			(xy 113.03 173.99) (xy 113.03 176.53)
 		)
 		(stroke
@@
 	(wire
 		(pts
-			(xy 95.25 187.96) (xy 92.71 187.96)
+			(xy 113.03 186.69) (xy 110.49 186.69)
 		)
 		(stroke
@@
 	(wire
 		(pts
-			(xy 101.6 182.88) (xy 92.71 182.88)
+			(xy 119.38 181.61) (xy 110.49 181.61)
 		)
 		(stroke
@@
 	(wire
 		(pts
-			(xy 71.12 187.96) (xy 80.01 187.96)
+			(xy 88.9 186.69) (xy 97.79 186.69)
 		)
 		(stroke
@@
 	(wire
 		(pts
-			(xy 71.12 185.42) (xy 80.01 185.42)
+			(xy 88.9 184.15) (xy 97.79 184.15)
 		)
 		(stroke
@@
 	(wire
 		(pts
-			(xy 101.6 185.42) (xy 92.71 185.42)
+			(xy 119.38 184.15) (xy 110.49 184.15)
 		)
 		(stroke
@@
 	)
 	(label "RX_PICO"
-		(at 101.6 185.42 180)
+		(at 119.38 184.15 180)
 		(effects
 			(font
@@
 	)
 	(label "MISO"
-		(at 71.12 180.34 0)
+		(at 88.9 179.07 0)
 		(effects
 			(font
@@
 	)
 	(label "USR0"
-		(at 71.12 187.96 0)
+		(at 88.9 186.69 0)
 		(effects
 			(font
@@
 	)
 	(label "SCK"
-		(at 71.12 182.88 0)
+		(at 88.9 181.61 0)
 		(effects
 			(font
@@
 	)
 	(label "TX_PICO"
-		(at 101.6 182.88 180)
+		(at 119.38 181.61 180)
 		(effects
 			(font
@@
 	)
 	(label "CS0"
-		(at 71.12 185.42 0)
+		(at 88.9 184.15 0)
 		(effects
 			(font
@@
 	)
 	(label "MOSI"
-		(at 71.12 177.8 0)
+		(at 88.9 176.53 0)
 		(effects
 			(font
@@
 	(symbol
 		(lib_id "power:+3.3V")
-		(at 102.87 175.26 0)
+		(at 120.65 173.99 0)
 		(unit 1)
 		(exclude_from_sim no)
@@
 		(fields_autoplaced yes)
 		(property "Reference" "#PWR021"
-			(at 102.87 179.07 0)
+			(at 120.65 177.8 0)
 			(effects
 				(font
@@
 		)
 		(property "Value" "+3.3V"
-			(at 102.87 170.18 0)
+			(at 120.65 168.91 0)
 			(effects
 				(font
@@
 		)
 		(property "Footprint" ""
-			(at 102.87 175.26 0)
+			(at 120.65 173.99 0)
 			(effects
 				(font
@@
 		)
 		(property "Datasheet" ""
-			(at 102.87 175.26 0)
+			(at 120.65 173.99 0)
 			(effects
 				(font
@@
 		)
 		(property "Description" "Power symbol creates a global label with name \"+3.3V\""
-			(at 102.87 175.26 0)
+			(at 120.65 173.99 0)
 			(effects
 				(font
@@
 	(symbol
 		(lib_id "power:GND")
-		(at 95.25 190.5 0)
+		(at 113.03 189.23 0)
 		(unit 1)
 		(exclude_from_sim no)
@@
 		(fields_autoplaced yes)
 		(property "Reference" "#PWR017"
-			(at 95.25 196.85 0)
+			(at 113.03 195.58 0)
 			(effects
 				(font
@@
 		)
 		(property "Value" "GND"
-			(at 95.25 195.58 0)
+			(at 113.03 194.31 0)
 			(effects
 				(font
@@
 		)
 		(property "Footprint" ""
-			(at 95.25 190.5 0)
+			(at 113.03 189.23 0)
 			(effects
 				(font
@@
 		)
 		(property "Datasheet" ""
-			(at 95.25 190.5 0)
+			(at 113.03 189.23 0)
 			(effects
 				(font
@@
 		)
 		(property "Description" "Power symbol creates a global label with name \"GND\" , ground"
-			(at 95.25 190.5 0)
+			(at 113.03 189.23 0)
 			(effects
 				(font
@@
 	(symbol
 		(lib_id "power:+5V")
-		(at 95.25 175.26 0)
+		(at 113.03 173.99 0)
 		(unit 1)
 		(exclude_from_sim no)
@@
 		(fields_autoplaced yes)
 		(property "Reference" "#PWR020"
-			(at 95.25 179.07 0)
+			(at 113.03 177.8 0)
 			(effects
 				(font
@@
 		)
 		(property "Value" "+5V"
-			(at 95.25 170.18 0)
+			(at 113.03 168.91 0)
 			(effects
 				(font
@@
 		)
 		(property "Footprint" ""
-			(at 95.25 175.26 0)
+			(at 113.03 173.99 0)
 			(effects
 				(font
@@
 		)
 		(property "Datasheet" ""
-			(at 95.25 175.26 0)
+			(at 113.03 173.99 0)
 			(effects
 				(font
@@
 		)
 		(property "Description" "Power symbol creates a global label with name \"+5V\""
-			(at 95.25 175.26 0)
+			(at 113.03 173.99 0)
 			(effects
 				(font
@@
 	(symbol
 		(lib_id "Connector_Generic:Conn_02x05_Counter_Clockwise")
-		(at 85.09 182.88 0)
+		(at 102.87 181.61 0)
 		(unit 1)
 		(exclude_from_sim no)
@@
 		(fields_autoplaced yes)
 		(property "Reference" "J6"
-			(at 86.36 171.45 0)
+			(at 104.14 170.18 0)
 			(effects
 				(font
@@
 		)
 		(property "Value" "External"
-			(at 86.36 173.99 0)
+			(at 104.14 172.72 0)
 			(effects
 				(font
@@
 		)
 		(property "Footprint" ""
-			(at 85.09 182.88 0)
+			(at 102.87 181.61 0)
 			(effects
 				(font
@@
 		)
 		(property "Datasheet" "~"
-			(at 85.09 182.88 0)
+			(at 102.87 181.61 0)
 			(effects
 				(font
@@
 		)
 		(property "Description" "Generic connector, double row, 02x05, counter clockwise pin numbering scheme (similar to DIP package numbering), script generated (kicad-library-utils/schlib/autogen/connector/)"
-			(at 85.09 182.88 0)
+			(at 102.87 181.61 0)
 			(effects
 				(font

Commit message: .
Connections:
- net MISO: now also A1.5 (GPIO3); no longer A1.6 (GPIO4)
- net MOSI: now also A1.6 (GPIO4); no longer A1.5 (GPIO3)
Other:
- note added: "These two are inverted ------> on pourpose"
Changed lines of the file:
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@@
+		)
+	)
+	(text "These two\nare inverted ------>\non pourpose"
+		(exclude_from_sim no)
+		(at 66.802 91.694 0)
+		(effects
+			(font
+				(size 1.27 1.27)
+			)
+			(justify left)
 		)
 	)
@@
 		)
 	)
-	(label "MISO"
+	(label "MOSI"
 		(at 91.44 93.98 0)
 		(effects
@@
 		)
 	)
-	(label "MOSI"
+	(label "MISO"
 		(at 91.44 91.44 0)
 		(effects
