File: schematic/pi-pico-vga.kicad_sch (KiCad schematic)
At the start: 33 parts, among them J1 VGA, J2 USB Keyboard, J3 Micro_SD_Card, J4 Power, J5 UART, J6 External, J7 Jack-DC, SW1 Power switch, SW2 User, SW3 Microswitch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

Commit message: .
Parts:
- removed J7: Jack-DC, symbol Connector:Jack-DC
- added J8: AudioJack4, symbol Connector_Audio:AudioJack4
Connections:
- net GND: now also J8.R2, J8.S
- net at C2.2: now also J8.R1, J8.T
Changed lines of the file:
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@@
 	)
 	(junction
+		(at 248.92 46.99)
+		(diameter 0)
+		(color 0 0 0 0)
+	)
+	(junction
 		(at 185.42 116.84)
 		(diameter 0)
@@
 	)
 	(junction
+		(at 248.92 41.91)
+		(diameter 0)
+		(color 0 0 0 0)
+	)
+	(junction
 		(at 34.29 59.69)
 		(diameter 0)
@@
 	(wire
 		(pts
+			(xy 248.92 41.91) (xy 248.92 39.37)
+		)
+		(stroke
+			(width 0)
+			(type default)
+		)
+	)
+	(wire
+		(pts
 			(xy 143.51 20.32) (xy 143.51 22.86)
 		)
@@
 	(wire
 		(pts
-			(xy 243.84 41.91) (xy 246.38 41.91)
+			(xy 243.84 41.91) (xy 248.92 41.91)
 		)
 		(stroke
@@
 	(wire
 		(pts
-			(xy 227.33 46.99) (xy 246.38 46.99)
+			(xy 227.33 46.99) (xy 248.92 46.99)
 		)
 		(stroke
@@
 	(wire
 		(pts
+			(xy 248.92 39.37) (xy 251.46 39.37)
+		)
+		(stroke
+			(width 0)
+			(type default)
+		)
+	)
+	(wire
+		(pts
 			(xy 148.59 93.98) (xy 170.18 93.98)
 		)
@@
 	(wire
 		(pts
+			(xy 248.92 41.91) (xy 251.46 41.91)
+		)
+		(stroke
+			(width 0)
+			(type default)
+		)
+	)
+	(wire
+		(pts
 			(xy 105.41 44.45) (xy 102.87 44.45)
 		)
@@
 	(wire
 		(pts
+			(xy 248.92 46.99) (xy 251.46 46.99)
+		)
+		(stroke
+			(width 0)
+			(type default)
+		)
+	)
+	(wire
+		(pts
 			(xy 43.18 130.81) (xy 43.18 119.38)
 		)
@@
 	(wire
 		(pts
+			(xy 248.92 44.45) (xy 248.92 46.99)
+		)
+		(stroke
+			(width 0)
+			(type default)
+		)
+	)
+	(wire
+		(pts
 			(xy 163.83 43.18) (xy 163.83 36.83)
 		)
@@
 	(wire
 		(pts
+			(xy 251.46 44.45) (xy 248.92 44.45)
+		)
+		(stroke
+			(width 0)
+			(type default)
+		)
+	)
+	(wire
+		(pts
 			(xy 26.67 59.69) (xy 34.29 59.69)
 		)
@@
 	)
 	(symbol
+		(lib_id "Connector_Audio:AudioJack4")
+		(at 256.54 44.45 180)
+		(unit 1)
+		(exclude_from_sim no)
+		(in_bom yes)
+		(on_board yes)
+		(dnp no)
+		(property "Reference" "J8"
+			(at 265.43 43.8151 0)
+			(effects
+				(font
+					(size 1.27 1.27)
+				)
+				(justify right)
+			)
+		)
+		(property "Value" "AudioJack4"
+			(at 265.43 41.2751 0)
+			(effects
+				(font
+					(size 1.27 1.27)
+				)
+				(justify right)
+			)
+		)
+		(property "Footprint" ""
+			(at 256.54 44.45 0)
+			(effects
+				(font
+					(size 1.27 1.27)
+				)
+				(hide yes)
+			)
+		)
+		(property "Datasheet" "~"
+			(at 256.54 44.45 0)
+			(effects
+				(font
+					(size 1.27 1.27)
+				)
+				(hide yes)
+			)
+		)
+		(property "Description" "Audio Jack, 4 Poles (TRRS)"
+			(at 256.54 44.45 0)
+			(effects
+				(font
+					(size 1.27 1.27)
+				)
+				(hide yes)
+			)
+		)
+		(pin "T"
+		)
+		(pin "S"
+		)
+		(pin "R1"
+		)
+		(pin "R2"
+		)
+		(instances
+			(project ""
+				(path "/b5f02af8-4b5a-49cc-8261-5c107f019f6d"
+					(reference "J8")
+					(unit 1)
+				)
+			)
+		)
+	)
+	(symbol
 		(lib_id "Device:R")
 		(at 173.99 91.44 90)
@@
 					(unit 1)
 				)
-			)
-		)
-	)
-	(symbol
-		(lib_id "Connector:Jack-DC")
-		(at 254 44.45 0)
-		(mirror y)
-		(unit 1)
-		(exclude_from_sim no)
-		(in_bom yes)
-		(on_board yes)
-		(dnp no)
-		(fields_autoplaced yes)
-		(property "Reference" "J7"
-			(at 260.35 43.1799 0)
-			(effects
-				(font
-					(size 1.27 1.27)
-				)
-				(justify right)
-			)
-		)
-		(property "Value" "Jack-DC"
-			(at 260.35 45.7199 0)
-			(effects
-				(font
-					(size 1.27 1.27)
-				)
-				(justify right)
-			)
-		)
-		(property "Footprint" ""
-			(at 252.73 45.466 0)
-			(effects
-				(font
-					(size 1.27 1.27)
-				)
-				(hide yes)
-			)
-		)
-		(property "Datasheet" "~"
-			(at 252.73 45.466 0)
-			(effects
-				(font
-					(size 1.27 1.27)
-				)
-				(hide yes)
-			)
-		)
-		(property "Description" "DC Barrel Jack"
-			(at 254 44.45 0)
-			(effects
-				(font
-					(size 1.27 1.27)
-				)
-				(hide yes)
-			)
-		)
-		(pin "1"
-		)
-		(pin "2"
-		)
-		(instances
-			(project ""
-				(path "/b5f02af8-4b5a-49cc-8261-5c107f019f6d"
-					(reference "J7")
-					(unit 1)
-				)
